Commit message: build and configure the moveit package for the robot

File: arduinobot_ws/src/arduinobot_description/urdf/arduinobot.urdf.xacro (robot description, xacro)
@@ -1,12 +1,33 @@
 <?xml version="1.0"?>
-<robot name="arduinobot" xmlns:xacro = "http://www.ros.org/wiki/xacro">
-    <!--Useful Variable (Properties)-->
-        <!-- Useful Variables (Properties) -->
+<robot xmlns:xacro="http://www.ros.org/wiki/xacro" name="arduinobot">
+    <!-- Useful Variables (Properties) -->
     <xacro:property name="PI" value="3.14159265359" />
     <xacro:property name="effort" value="30" />
     <xacro:property name="velocity" value="10" />
+    <!-- Useful Macros -->
+    <xacro:macro name="default_inertial" params="mass">
+        <inertial>
+            <mass value="${mass}" />
+            <inertia ixx="1.0" ixy="0.0" ixz="0.0"
+                     iyy="1.0" iyz="0.0"
+                     izz="1.0" />
+        </inertial>
+    </xacro:macro>
+    <xacro:macro name="default_transmission" params="number">
+        <transmission name="transmission_${number}">
+            <type>transmission_interface/SimpleTransmission</type>
+            <joint name="joint_${number}">
+                <hardwareInterface>hardware_interface/PositionJointInterface</hardwareInterface>
+            </joint>
+            <actuator name="motor_${number}">
+                <hardwareInterface>hardware_interface/PositionJointInterface</hardwareInterface>
+                <mechanicalReduction>1</mechanicalReduction>
+            </actuator>
+        </transmission>
+    </xacro:macro>
     <!-- Links -->
-    <link name = "world" />
-        <link name="base_link">
+    <link name="world"/>
+    <link name="base_link">
+        <xacro:default_inertial mass="1"/>
         <visual>
             <origin rpy="0 0 0" xyz="-0.5 -0.5 0"/>
@@ -18,8 +39,18 @@
             </material>
         </visual>
+        <collision>
+            <origin rpy="0 0 0" xyz="-0.5 -0.5 0"/>
+            <geometry>
+                <mesh filename="package://arduinobot_description/mesh/basement.STL" scale="0.01 0.01 0.01"/>
+            </geometry>
+            <material name="bluish" >
+                <color rgba="0.1607843137254902 0.4627450980392157 0.7333333333333333 1.0" />
+            </material>
+        </collision>
     </link>
     <link name="base_plate">
-        <visual>
-            <origin rpy="0 0 0" xyz="-0.35 -0.39 -0.56"/>
+        <xacro:default_inertial mass="0.1"/>
+        <visual>
+            <origin rpy="0 0 0" xyz="-0.39 -0.39 -0.56"/>
             <geometry>
                 <mesh filename="package://arduinobot_description/mesh/base_plate.STL" scale="0.01 0.01 0.01"/>
@@ -29,6 +60,16 @@
             </material>
         </visual>
+        <collision>
+            <origin rpy="0 0 0" xyz="-0.39 -0.39 -0.56"/>
+            <geometry>
+                <mesh filename="package://arduinobot_description/mesh/base_plate.STL" scale="0.01 0.01 0.01"/>
+            </geometry>
+            <material name="bluish" >
+                <color rgba="0.1607843137254902 0.4627450980392157 0.7333333333333333 1.0" />
+            </material>
+        </collision>
     </link>
     <link name="forward_drive_arm">
+        <xacro:default_inertial mass="0.1"/>
         <visual>
             <origin rpy=" 0 -${PI/2} ${PI/2}" xyz="0.19 0.06 -0.08"/>
@@ -40,6 +81,16 @@
             </material>
         </visual>
+        <collision>
+            <origin rpy=" 0 -${PI/2} ${PI/2}" xyz="0.19 0.06 -0.08"/>
+            <geometry>
+                <mesh filename="package://arduinobot_description/mesh/forward_drive_arm.STL" scale="0.01 0.01 0.01"/>
+            </geometry>
+            <material name="bluish" >
+                <color rgba="0.1607843137254902 0.4627450980392157 0.7333333333333333 1.0" />
+            </material>
+        </collision>
     </link>
     <link name="horizontal_arm">
+        <xacro:default_inertial mass="0.1"/>
         <visual>
             <origin rpy="${PI/2} 0 ${PI/2}" xyz="-0.03 -0.4 -0.06"/>
@@ -51,6 +102,16 @@
             </material>
         </visual>
+        <collision>
+            <origin rpy="${PI/2} 0 ${PI/2}" xyz="-0.03 -0.4 -0.06"/>
+            <geometry>
+                <mesh filename="package://arduinobot_description/mesh/horizontal_arm.STL" scale="0.01 0.01 0.01"/>
+            </geometry>
+            <material name="bluish" >
+                <color rgba="0.1607843137254902 0.4627450980392157 0.7333333333333333 1.0" />
+            </material>
+        </collision>
     </link>
     <link name="claw_support">
+        <xacro:default_inertial mass="0.05"/>
         <visual>
             <origin rpy="0 0 ${PI/2}" xyz="0 -0.05 -0.15"/>
@@ -62,6 +123,16 @@
             </material>
         </visual>
+        <collision>
+            <origin rpy="0 0 ${PI/2}" xyz="0 -0.05 -0.15"/>
+            <geometry>
+                <mesh filename="package://arduinobot_description/mesh/claw_support.STL" scale="0.01 0.01 0.01"/>
+            </geometry>
+            <material name="bluish" >
+                <color rgba="0.1607843137254902 0.4627450980392157 0.7333333333333333 1.0" />
+            </material>
+        </collision>
     </link>
     <link name="gripper_right">
+        <xacro:default_inertial mass="0.01"/>
         <visual>
             <origin rpy="0 0 -${PI/2}" xyz="-0.1 0.50 -0.1"/>
@@ -73,6 +144,16 @@
             </material>
         </visual>
+        <collision>
+            <origin rpy="0 0 -${PI/2}" xyz="-0.1 0.50 -0.1"/>
+            <geometry>
+                <mesh filename="package://arduinobot_description/mesh/right_finger.STL" scale="0.01 0.01 0.01"/>
+            </geometry>
+            <material name="bronze" >
+                <color rgba="0.6588235294117647 0.4745098039215686 0.0 1.0" />
+            </material>
+        </collision>
     </link>
     <link name="gripper_left">
+        <xacro:default_inertial mass="0.01"/>
         <visual>
             <origin rpy="0 0 -${PI/2}" xyz="-0.04 0.50 -0.1"/>
@@ -84,4 +165,13 @@
             </material>
         </visual>
+        <collision>
+            <origin rpy="0 0 -${PI/2}" xyz="-0.04 0.50 -0.1"/>
+            <geometry>
+                <mesh filename="package://arduinobot_description/mesh/left_finger.STL" scale="0.01 0.01 0.01"/>
+            </geometry>
+            <material name="bronze" >
+                <color rgba="0.6588235294117647 0.4745098039215686 0.0 1.0" />
+            </material>
+        </collision>
     </link>
     <link name="tool_link"></link>
@@ -90,14 +180,14 @@
         <parent link="world"/>
         <child link="base_link"/>
-        <origin rpy="0.0 0.0 0.0" xyz="0.0 0.0 0.0"/>
-    </joint>
-    <joint name="joint_1" type="revolute">
+        <origin xyz="0 0 0" rpy="0 0 0"/>
+    </joint>
+    <joint name ="joint_1" type="revolute">
         <parent link="base_link"/>
-        <child link="base_plate"/>
-        <origin xyz="0.0 0.0 0.307"/>
-        <axis xyz="0.0 0.0 1"/>
+        <child link = "base_plate"/>
+        <origin xyz="0 0 0.307"/>
+        <axis xyz="0 0 1"/>
         <limit lower="-${PI/2}" upper="${PI/2}" effort="${effort}" velocity="${velocity}"/>
     </joint>
-        <joint name ="joint_2" type="revolute">
+    <joint name ="joint_2" type="revolute">
         <parent link="base_plate"/>
         <child link = "forward_drive_arm"/>
@@ -138,3 +228,24 @@
         <origin xyz="0 0 0"/>
     </joint>
+    <!-- Transmissions-->
+    <xacro:default_transmission number="1"/>
+    <xacro:default_transmission number="2"/>
+    <xacro:default_transmission number="3"/>
+    <xacro:default_transmission number="4"/>
+    <!-- gazebo ros_control plugin -->
+    <gazebo>
+        <plugin name="gazebo_ros_control" filename="libgazebo_ros_control.so">
+            <robotNamespace>/arduinobot</robotNamespace>
+            <robotSimType>gazebo_ros_control/DefaultRobotHWSim</robotSimType>
+            <legacyModeNS>true</legacyModeNS>
+        </plugin>
+        <plugin name="joint_5_mimic_joint_4" filename="libroboticsgroup_upatras_gazebo_mimic_joint_plugin.so">
+          <joint>joint_4</joint>
+          <mimicJoint>joint_5</mimicJoint>
+          <multiplier>-1.0</multiplier>
+          <offset>0</offset>
+          <maxEffort>${effort}</maxEffort>
+          <robotNamespace>/arduinobot</robotNamespace>
+        </plugin>
+    </gazebo>
 </robot>

Commit message: add controller and hardware interface - add moveit package and complete its configuration

File: arduinobot_ws/src/arduinobot_description/urdf/arduinobot.urdf.xacro (robot description, xacro)
@@ -5,20 +5,18 @@
     <xacro:property name="effort" value="30" />
     <xacro:property name="velocity" value="10" />
-    <!-- Useful Macros -->
-    <xacro:macro name="default_inertial" params="mass">
+    <!--Useful macro -->
+    <xacro:macro name ="default_inertial" params = "mass">
         <inertial>
-            <mass value="${mass}" />
-            <inertia ixx="1.0" ixy="0.0" ixz="0.0"
-                     iyy="1.0" iyz="0.0"
-                     izz="1.0" />
+            <mass value="${mass}"/>
+            <inertia ixx = "1" iyy = "1" izz = "1" ixy = "0" ixz = "0" iyz = "0" />
         </inertial>
     </xacro:macro>
-    <xacro:macro name="default_transmission" params="number">
-        <transmission name="transmission_${number}">
+    <xacro:macro name = "default_transmission" params = "number">
+        <transmission name = "joint_${number}">
             <type>transmission_interface/SimpleTransmission</type>
-            <joint name="joint_${number}">
+            <joint name = "joint_${number}">
                 <hardwareInterface>hardware_interface/PositionJointInterface</hardwareInterface>
             </joint>
-            <actuator name="motor_${number}">
+            <actuator name ="motor_${number}">
                 <hardwareInterface>hardware_interface/PositionJointInterface</hardwareInterface>
                 <mechanicalReduction>1</mechanicalReduction>
@@ -29,5 +27,5 @@
     <link name="world"/>
     <link name="base_link">
-        <xacro:default_inertial mass="1"/>
+        <xacro:default_inertial mass = "1"/>
         <visual>
             <origin rpy="0 0 0" xyz="-0.5 -0.5 0"/>
@@ -50,5 +48,5 @@
     </link>
     <link name="base_plate">
-        <xacro:default_inertial mass="0.1"/>
+        <xacro:default_inertial mass = "0.1"/>
         <visual>
             <origin rpy="0 0 0" xyz="-0.39 -0.39 -0.56"/>
@@ -61,4 +59,5 @@
         </visual>
         <collision>
+            <xacro:default_inertial mass = "0.1"/>
             <origin rpy="0 0 0" xyz="-0.39 -0.39 -0.56"/>
             <geometry>
@@ -71,5 +70,5 @@
     </link>
     <link name="forward_drive_arm">
-        <xacro:default_inertial mass="0.1"/>
+        <xacro:default_inertial mass = "0.1"/>
         <visual>
             <origin rpy=" 0 -${PI/2} ${PI/2}" xyz="0.19 0.06 -0.08"/>
@@ -92,5 +91,5 @@
     </link>
     <link name="horizontal_arm">
-        <xacro:default_inertial mass="0.1"/>
+        <xacro:default_inertial mass = "0.1"/>
         <visual>
             <origin rpy="${PI/2} 0 ${PI/2}" xyz="-0.03 -0.4 -0.06"/>
@@ -113,5 +112,5 @@
     </link>
     <link name="claw_support">
-        <xacro:default_inertial mass="0.05"/>
+        <xacro:default_inertial mass = "0.05"/>
         <visual>
             <origin rpy="0 0 ${PI/2}" xyz="0 -0.05 -0.15"/>
@@ -134,5 +133,5 @@
     </link>
     <link name="gripper_right">
-        <xacro:default_inertial mass="0.01"/>
+        <xacro:default_inertial mass = "0.01"/>
         <visual>
             <origin rpy="0 0 -${PI/2}" xyz="-0.1 0.50 -0.1"/>
@@ -155,6 +154,6 @@
     </link>
     <link name="gripper_left">
-        <xacro:default_inertial mass="0.01"/>
-        <visual>
+        <visual>
+            <xacro:default_inertial mass = "0.01"/>
             <origin rpy="0 0 -${PI/2}" xyz="-0.04 0.50 -0.1"/>
             <geometry>
@@ -228,10 +227,10 @@
         <origin xyz="0 0 0"/>
     </joint>
-    <!-- Transmissions-->
-    <xacro:default_transmission number="1"/>
-    <xacro:default_transmission number="2"/>
-    <xacro:default_transmission number="3"/>
-    <xacro:default_transmission number="4"/>
-    <!-- gazebo ros_control plugin -->
+    <!--Joint_transmission-->
+    <xacro:default_transmission number = "1"/>
+    <xacro:default_transmission number = "2"/>
+    <xacro:default_transmission number = "3"/>
+    <xacro:default_transmission number = "4"/>
+    <!--gazebo ros_control plugin -->
     <gazebo>
         <plugin name="gazebo_ros_control" filename="libgazebo_ros_control.so">
@@ -240,11 +239,12 @@
             <legacyModeNS>true</legacyModeNS>
         </plugin>
-        <plugin name="joint_5_mimic_joint_4" filename="libroboticsgroup_upatras_gazebo_mimic_joint_plugin.so">
-          <joint>joint_4</joint>
-          <mimicJoint>joint_5</mimicJoint>
-          <multiplier>-1.0</multiplier>
-          <offset>0</offset>
-          <maxEffort>${effort}</maxEffort>
-          <robotNamespace>/arduinobot</robotNamespace>
+    <!-- gazebo_mimic_joint_plugin -->
+        <plugin name = "joint_5_mimic_joint_4" filename = "libroboticsgroup_upatras_gazebo_mimic_joint_plugin.so">
+            <joint>joint_4</joint>
+            <mimicJoint>joint_5</mimicJoint>
+            <multiplier>-1.0</multiplier>
+            <offset>0</offset>
+            <maxEffort>${effort}</maxEffort>
+            <robotNamespace>/arduinobot</robotNamespace>
         </plugin>
     </gazebo>
